Commit message: Spot lidar and gmapping

File: src/spot_ros/spot_description/urdf/accessories.urdf.xacro (robot description, xacro)
@@ -1,74 +1,68 @@
 <?xml version="1.0"?>
 <robot xmlns:xacro="http://www.ros.org/wiki/xacro">
-  <xacro:if value="$(optenv SPOT_PACK 0)">
-    <joint name="pack_mount_joint" type="fixed">
-      <parent link="base_link"/>
-      <child link="pack_mount"/>
-      <origin xyz="-0.019986 0 0.093662" rpy="0 0 0"/>
-    </joint>
-    <link name="pack_mount">
-      <visual>
-        <geometry>
-          <mesh filename="package://spot_description/meshes/pack_top.dae"/>
-        </geometry>
-      </visual>
-      <visual>
-        <geometry>
-          <mesh filename="package://spot_description/meshes/pack_body.dae"/>
-        </geometry>
-      </visual>
-      <collision>
-        <geometry>
-          <mesh filename="package://spot_description/meshes/pack_body.dae"/>
-        </geometry>
-      </collision>
-    </link>
-  </xacro:if>
-  <xacro:if value="$(optenv SPOT_LIDAR_MOUNT 0)">
-    <joint name="lidar_mount_joint" type="fixed">
-      <parent link="pack_mount"/>
-      <child link="lidar_mount"/>
-      <origin xyz="0.015 0 0.149285" rpy="0 0 0"/>
-    </joint>
-    <link name="lidar_mount">
-      <visual>
-        <geometry>
-          <mesh filename="package://spot_description/meshes/lidar_mount.dae"/>
-        </geometry>
-      </visual>
-      <collision>
-        <geometry>
-          <mesh filename="package://spot_description/meshes/lidar_mount_collision.stl"/>
-        </geometry>
-      </collision>
-    </link>
-    <xacro:if value="$(optenv SPOT_VELODYNE 0)">
-      <!-- Use the Velodyne macro for the actual sensor -->
-      <xacro:include filename="$(find velodyne_description)/urdf/VLP-16.urdf.xacro" />
-      <xacro:VLP-16 parent="lidar_mount">
-        <origin xyz="$(optenv SPOT_VELODYNE_XYZ 0 0 0)" rpy="$(optenv SPOT_VELODYNE_RPY 0 0 0)" />
-      </xacro:VLP-16>
-      <!-- Add the protective cage -->
-      <link name="velodyne_cage">
-        <visual>
-          <geometry>
-            <mesh filename="package://spot_description/meshes/velodyne_cage.stl" scale="0.001 0.001 0.001" />
-          </geometry>
-          <origin xyz="0 0 0" rpy="0 0 0" />
-          <material name="black" />
-        </visual>
-        <collision>
-          <geometry>
-            <mesh filename="package://spot_description/meshes/velodyne_cage.stl" scale="0.001 0.001 0.001" />
-          </geometry>
-          <origin xyz="0 0 0" rpy="0 0 0" />
-        </collision>
-      </link>
-      <joint name="velodyne_cage_joint" type="fixed">
-        <parent link="lidar_mount" />
-        <child link="velodyne_cage" />
-        <origin xyz="$(optenv SPOT_VELODYNE_XYZ 0 0 0)" rpy="$(optenv SPOT_VELODYNE_RPY 0 0 0)" />
-      </joint>
-    </xacro:if>
-  </xacro:if>
+  <joint name="pack_mount_joint" type="fixed">
+    <parent link="base_link" />
+    <child link="pack_mount" />
+    <origin xyz="-0.019986 0 0.093662" rpy="0 0 0" />
+  </joint>
+  <link name="pack_mount">
+    <visual>
+      <geometry>
+        <mesh filename="package://spot_description/meshes/pack_top.dae" />
+      </geometry>
+    </visual>
+    <visual>
+      <geometry>
+        <mesh filename="package://spot_description/meshes/pack_body.dae" />
+      </geometry>
+    </visual>
+    <collision>
+      <geometry>
+        <mesh filename="package://spot_description/meshes/pack_body.dae" />
+      </geometry>
+    </collision>
+  </link>
+  <joint name="lidar_mount_joint" type="fixed">
+    <parent link="pack_mount" />
+    <child link="lidar_mount" />
+    <origin xyz="0.015 0 0.149285" rpy="0 0 0" />
+  </joint>
+  <link name="lidar_mount">
+    <visual>
+      <geometry>
+        <mesh filename="package://spot_description/meshes/lidar_mount.dae" />
+      </geometry>
+    </visual>
+    <collision>
+      <geometry>
+        <mesh filename="package://spot_description/meshes/lidar_mount_collision.stl" />
+      </geometry>
+    </collision>
+  </link>
+  <!-- Use the Velodyne macro for the actual sensor -->
+  <xacro:include filename="$(find velodyne_description)/urdf/VLP-16.urdf.xacro" />
+  <xacro:VLP-16 parent="lidar_mount">
+    <origin xyz="$(optenv SPOT_VELODYNE_XYZ 0 0 0)" rpy="$(optenv SPOT_VELODYNE_RPY 0 0 0)" />
+  </xacro:VLP-16>
+  <!-- Add the protective cage -->
+  <link name="velodyne_cage">
+    <visual>
+      <geometry>
+        <mesh filename="package://spot_description/meshes/velodyne_cage.stl" scale="0.001 0.001 0.001" />
+      </geometry>
+      <origin xyz="0 0 0" rpy="0 0 0" />
+      <material name="black" />
+    </visual>
+    <collision>
+      <geometry>
+        <mesh filename="package://spot_description/meshes/velodyne_cage.stl" scale="0.001 0.001 0.001" />
+      </geometry>
+      <origin xyz="0 0 0" rpy="0 0 0" />
+    </collision>
+  </link>
+  <joint name="velodyne_cage_joint" type="fixed">
+    <parent link="lidar_mount" />
+    <child link="velodyne_cage" />
+    <origin xyz="$(optenv SPOT_VELODYNE_XYZ 0 0 0)" rpy="$(optenv SPOT_VELODYNE_RPY 0 0 0)" />
+  </joint>
 </robot>
