Commit message: move_base and description launch files

File: src/spot_pkg/spot_description/urdf/accessories.urdf.xacro (robot description, xacro)
@@ -1,84 +1,66 @@
 <?xml version="1.0"?>
 <robot xmlns:xacro="http://www.ros.org/wiki/xacro">
-  <joint name="ny_lidar_mount_joint" type="fixed">
+  <!-- Forward Mount -->
+  <joint name="lidar_mount_forward_joint" type="fixed">
     <parent link="base_link" />
-    <child link="ny_lidar_mount" />
-    <origin xyz="0 0.5 0.06" rpy="0 0 0" />
+    <child link="lidar_mount_forward" />
+    <origin xyz="0.1 -0.097 0.075" rpy="1.57 0 1.57" /> <!-- x: Forward/Back, y: Left/Right, z: Up/Down-->
   </joint>
-  <link name="ny_lidar_mount">
+  <link name="lidar_mount_forward">
     <visual>
       <geometry>
-        <mesh filename="package://spot_description/meshes/Spot_TOP.stl" />
+        <mesh filename="package://spot_pkg/spot_description/meshes/Spot_Top.stl" scale="0.0009 0.0009 0.0009" />
       </geometry>
+      <material name="Material_Color">
+        <color rgba="1.0 1.0 1.0 1.0"/>
+      </material>
     </visual>
     <collision>
       <geometry>
-        <mesh filename="package://spot_description/meshes/Spot_TOP.stl" />
+        <mesh filename="package://spot_pkg/spot_description/meshes/Spot_Top.stl" />
       </geometry>
     </collision>
   </link>
-  <xacro:macro name="sick_tim551" params="name ros_topic min_angle:=-2.357 max_angle:=2.357 min_range:=0.05 max_range:=10">
-    <xacro:sick_tim name="${name}" ros_topic="${ros_topic}"
-      length="0.06" width="0.06" height="0.086" mass="0.250" z_offset="0.06296"
-      min_range="${min_range}" max_range="${max_range}"
-      min_angle="${min_angle}" max_angle="${max_angle}"
-      mesh="package://sick_tim/meshes/sick_tim551.stl" />
-  </xacro:macro>
-  <xacro:macro name="sick_tim" params="name ros_topic length width height mass z_offset min_angle max_angle min_range max_range mesh">
-    <!-- z_offset: distance between base plate and laser center (= center of mesh) -->
-    <joint name="$sick_tim_joint" type="fixed">
-      <parent link="ny_lidar_mount" />
-      <child link="sick_tim" />
-      <origin rpy="0 0 0" xyz="0 0.06 0.03"/>
-    </joint>
-    <link name="sick_tim">
-      <visual>
-        <geometry>
-          <mesh filename="${mesh}" />
-        </geometry>
-        <material name="blue" >
-          <color rgba="0 0 1 1" />
-        </material>
-      </visual>
-      <collision>
-        <geometry>
-          <mesh filename="${mesh}" />
-        </geometry>
-      </collision>
-      <inertial>
-        <mass value="${mass}" />
-        <origin xyz="0 0 -0.026" />
-        <inertia ixx="${0.0833333 * mass * (width * width + height * height)}" ixy="0.0" ixz="0.0"
-          iyy="${0.0833333 * mass * (length * length + height * height)}" iyz="0.0"
-          izz="${0.0833333 * mass * (length * length + width * width)}" />
-      </inertial>
-    </link>
-  </xacro:macro>
-  <!-- Use the Velodyne macro for the actual sensor -->
-<!--   <xacro:include filename="$(find velodyne_description)/urdf/VLP-16.urdf.xacro" />
-  <xacro:VLP-16 parent="lidar_mount">
-    <origin xyz="$(optenv SPOT_VELODYNE_XYZ 0 0 0)" rpy="$(optenv SPOT_VELODYNE_RPY 0 0 0)" />
-  </xacro:VLP-16>
- -->
-  <!-- Add the protective cage -->
-<!--   <link name="velodyne_cage">
+  <!-- Back Mount -->
+  <joint name="lidar_mount_back_joint" type="fixed">
+    <parent link="base_link" />
+    <child link="lidar_mount_back" />
+    <origin xyz="-0.05 -0.097 0.075" rpy="1.57 0 1.57" /> <!-- x: Forward/Back, y: Left/Right, z: Up/Down-->
+  </joint>
+  <link name="lidar_mount_back">
     <visual>
       <geometry>
-        <mesh filename="package://spot_description/meshes/velodyne_cage.stl" scale="0.001 0.001 0.001" />
+        <mesh filename="package://spot_pkg/spot_description/meshes/Spot_Top.stl" scale="0.0009 0.0009 0.0009" />
       </geometry>
-      <origin xyz="0 0 0" rpy="0 0 0" />
-      <material name="black" />
+      <material name="Material_Color">
+        <color rgba="1.0 1.0 1.0 1.0"/>
+      </material>
     </visual>
     <collision>
       <geometry>
-        <mesh filename="package://spot_description/meshes/velodyne_cage.stl" scale="0.001 0.001 0.001" />
+        <mesh filename="package://spot_pkg/spot_description/meshes/Spot_Top.stl" />
       </geometry>
-      <origin xyz="0 0 0" rpy="0 0 0" />
     </collision>
   </link>
-  <joint name="velodyne_cage_joint" type="fixed">
-    <parent link="lidar_mount" />
-    <child link="velodyne_cage" />
-    <origin xyz="$(optenv SPOT_VELODYNE_XYZ 0 0 0)" rpy="$(optenv SPOT_VELODYNE_RPY 0 0 0)" />
+  <!-- Sick tim Lidar -->
+  <joint name="sick_tim_joint" type="fixed">
+    <parent link="lidar_mount_forward" />
+    <child link="sick_tim" />
+    <origin rpy="-1.57 -1.57 0" xyz="0.1 0.12 0.09"/>
   </joint>
-</robot> -->
+  <link name="sick_tim">
+    <visual>
+      <geometry>
+        <mesh filename="package://sick_tim/meshes/sick_tim551.stl" />
+      </geometry>
+      <material name="grey" >
+        <color rgba="1 0.1 0.1 1.0" />
+      </material>
+    </visual>
+    <collision>
+      <geometry>
+        <mesh filename="package://sick_tim/meshes/sick_tim551.stl" />
+      </geometry>
+    </collision>
+  </link>
+</robot>

File: src/spot_pkg/spot_description/urdf/spot.urdf.xacro (robot description, xacro)
@@ -260,5 +260,5 @@
     </joint>
     <!-- Standard accessories. -->
-    <xacro:include filename="$(find spot_pkg)/urdf/accessories.urdf.xacro" />
+    <xacro:include filename="$(find spot_pkg)/spot_description/urdf/accessories.urdf.xacro" />
     <!-- Optional custom includes. -->
     <xacro:include filename="$(optenv SPOT_URDF_EXTRAS empty.urdf)" />
